File: Eagle/HAB1 Schematic.sch (EAGLE design)
At the start: 17 parts, among them U1 microSD

Commit message: Update
Parts:
- removed R6: 10K, rcl:R-EU_0204/5
- removed U1: microSD, SparkFun:USD-SOCKETSMD
- added A0: A0, wirepad:1,6/0,8
- added A1: A1, wirepad:1,6/0,8
- added A3: A3, wirepad:1,6/0,8
- added A6: A6, wirepad:1,6/0,8
- added A7: A7, wirepad:1,6/0,8
- added D4: D4, wirepad:1,6/0,8
- added D5: D5, wirepad:1,6/0,8
- added D6: D6, wirepad:1,6/0,8
- added D9: D9, wirepad:1,6/0,8
- added RST: RST, wirepad:1,6/0,8
- GRN, RED: value (none) -> LED
- JP1: value (none) -> SD
Connections:
- net CS renamed N$1
- net SCK renamed N$21
- removed net DI: ARDUINO.12, JP1.2
- removed net DO: ARDUINO.*11, JP1.6
- removed net N$1 (its old number): R6.1, U$3.TXD
- new net A0: A0.P, ARDUINO.A0
- new net A1: A1.P, ARDUINO.A1
- new net A3: A3.P, ARDUINO.A3
- new net A6: A6.P, ARDUINO.A6
- new net A7: A7.P, ARDUINO.A7
- new net D4: ARDUINO.4, D4.P
- new net D5: ARDUINO.*5, D5.P
- new net D6: ARDUINO.*6, D6.P
- new net D9: ARDUINO.*9, D9.P
- new net N$19: ARDUINO.12, JP1.6
- new net N$20: ARDUINO.*11, JP1.2
- new net RST: ARDUINO.RST, ARDUINO.RST@2, RST.P
- net GND: now also ARDUINO.GND
- net N$6: now also U$3.TXD; no longer R6.2
- net RAW: now also U$3.EN, U$3.VCC
- net VCC: no longer U$3.EN, U$3.VCC
Other:
- moved on the sheet: JP1, RF_ANT

Commit message: Updated PCB
Parts:
- removed A6: A6, wirepad:1,6/0,8
- removed A7: A7, wirepad:1,6/0,8
- added GND: GND, wirepad:1,6/0,8
- added RAW: RAW, wirepad:1,6/0,8
- added VCC: VCC, wirepad:1,6/0,8
- R1: value 100 -> 10K
- R2: value 50 -> 4K7
Connections:
- removed net A6: A6.P, ARDUINO.A6
- removed net A7: A7.P, ARDUINO.A7
- net GND: now also GND.P
- net RAW: now also RAW.P
- net RST: no longer ARDUINO.RST
- net VCC: now also VCC.P
Changed lines of the file:
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@@
 <parts>
 <part name="ARDUINO" library="SparkFun-Boards" deviceset="ARDUINO_PRO_MINI" device=""/>
-<part name="R1" library="rcl" deviceset="R-EU_" device="0204/5" value="100"/>
-<part name="R2" library="rcl" deviceset="R-EU_" device="0204/5" value="50"/>
+<part name="R1" library="rcl" deviceset="R-EU_" device="0204/5" value="10K"/>
+<part name="R2" library="rcl" deviceset="R-EU_" device="0204/5" value="4K7"/>
 <part name="R3" library="rcl" deviceset="R-EU_" device="0204/5" value="4K7"/>
 <part name="R4" library="rcl" deviceset="R-EU_" device="0204/5" value="58"/>
@@
 <part name="D6" library="wirepad" deviceset="1,6/0,8" device="" value="D6"/>
 <part name="D9" library="wirepad" deviceset="1,6/0,8" device="" value="D9"/>
-<part name="A7" library="wirepad" deviceset="1,6/0,8" device="" value="A7"/>
-<part name="A6" library="wirepad" deviceset="1,6/0,8" device="" value="A6"/>
 <part name="A0" library="wirepad" deviceset="1,6/0,8" device="" value="A0"/>
 <part name="A1" library="wirepad" deviceset="1,6/0,8" device="" value="A1"/>
 <part name="A3" library="wirepad" deviceset="1,6/0,8" device="" value="A3"/>
 <part name="RST" library="wirepad" deviceset="1,6/0,8" device="" value="RST"/>
+<part name="GND" library="wirepad" deviceset="1,6/0,8" device="" value="GND"/>
+<part name="VCC" library="wirepad" deviceset="1,6/0,8" device="" value="VCC"/>
+<part name="RAW" library="wirepad" deviceset="1,6/0,8" device="" value="RAW"/>
 </parts>
 <sheets>
@@
 <instance part="D6" gate="P" x="60.96" y="15.24"/>
 <instance part="D9" gate="P" x="60.96" y="10.16"/>
-<instance part="A7" gate="P" x="101.6" y="81.28"/>
-<instance part="A6" gate="P" x="101.6" y="76.2"/>
 <instance part="A0" gate="P" x="101.6" y="86.36"/>
 <instance part="A1" gate="P" x="101.6" y="91.44"/>
 <instance part="A3" gate="P" x="101.6" y="96.52"/>
 <instance part="RST" gate="P" x="60.96" y="5.08"/>
+<instance part="GND" gate="P" x="116.84" y="96.52"/>
+<instance part="VCC" gate="P" x="116.84" y="86.36"/>
+<instance part="RAW" gate="P" x="116.84" y="76.2"/>
 </instances>
 <busses>
@@
 <label x="99.06" y="38.1" size="1.778" layer="95" rot="R90" xref="yes"/>
 </segment>
+<segment>
+<pinref part="VCC" gate="P" pin="P"/>
+<wire x1="119.38" y1="86.36" x2="121.92" y2="86.36" width="0.1524" layer="91"/>
+<label x="121.92" y="86.36" size="1.778" layer="95" xref="yes"/>
+</segment>
 </net>
 <net name="GND" class="0">
@@
 <label x="50.8" y="71.12" size="1.778" layer="95" rot="R180" xref="yes"/>
 </segment>
+<segment>
+<pinref part="GND" gate="P" pin="P"/>
+<wire x1="119.38" y1="96.52" x2="121.92" y2="96.52" width="0.1524" layer="91"/>
+<label x="121.92" y="96.52" size="1.778" layer="95" xref="yes"/>
+</segment>
 </net>
 <net name="RAW" class="0">
@@
 <label x="17.78" y="25.4" size="1.778" layer="95" xref="yes"/>
 <pinref part="U$3" gate="G$1" pin="EN"/>
+</segment>
+<segment>
+<pinref part="RAW" gate="P" pin="P"/>
+<wire x1="119.38" y1="76.2" x2="121.92" y2="76.2" width="0.1524" layer="91"/>
+<label x="121.92" y="76.2" size="1.778" layer="95" xref="yes"/>
 </segment>
 </net>
@@
 </segment>
 </net>
-<net name="A7" class="0">
-<segment>
-<pinref part="A7" gate="P" pin="P"/>
-<wire x1="104.14" y1="81.28" x2="106.68" y2="81.28" width="0.1524" layer="91"/>
-<label x="106.68" y="81.28" size="1.778" layer="95" xref="yes"/>
-</segment>
-<segment>
-<pinref part="ARDUINO" gate="G$1" pin="A7"/>
-<wire x1="76.2" y1="40.64" x2="78.74" y2="40.64" width="0.1524" layer="91"/>
-<label x="78.74" y="40.64" size="1.778" layer="95" xref="yes"/>
-</segment>
-</net>
-<net name="A6" class="0">
-<segment>
-<pinref part="A6" gate="P" pin="P"/>
-<wire x1="104.14" y1="76.2" x2="106.68" y2="76.2" width="0.1524" layer="91"/>
-<label x="106.68" y="76.2" size="1.778" layer="95" xref="yes"/>
-</segment>
-<segment>
-<pinref part="ARDUINO" gate="G$1" pin="A6"/>
-<wire x1="76.2" y1="38.1" x2="78.74" y2="38.1" width="0.1524" layer="91"/>
-<label x="78.74" y="38.1" size="1.778" layer="95" xref="yes"/>
-</segment>
-</net>
 <net name="RST" class="0">
 <segment>
@@
 <label x="78.74" y="68.58" size="1.778" layer="95" xref="yes"/>
 </segment>
-<segment>
-<pinref part="ARDUINO" gate="G$1" pin="RST"/>
-<wire x1="53.34" y1="68.58" x2="50.8" y2="86.36" width="0.1524" layer="91"/>
-<label x="50.8" y="86.36" size="1.778" layer="95" rot="R180" xref="yes"/>
-</segment>
-</net>
+</net>
